File: KicadPower/PowerStage.kicad_sch (KiCad schematic)
At the start: 24 parts, among them Q1 IGB110S101, Q11 IGB110S101, Q14 IGB110S101, Q17 IGB110S101, Q20 IGB110S101, Q24 IGB110S101, Q5 IGB110S101, Q8 IGB110S101

Commit message: minor changes
Parts:
- renumbered C145 to C147, C148 to C150, C151 to C153, C155 to C156, C159 to C157, C161 to C162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
Other:
- moved on the sheet: C147, C150, C153, C156, C157, C162, C164, C168, Q11, Q14, Q17, Q2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
