File: KicadPower/Sensing.kicad_sch (KiCad schematic)
At the start: 11 parts, among them P3 PIN 2, U2 TLE4972-AE35S5

Commit message: minor changes
Parts:
- renumbered C174 to C169, C169 to C173, C175 to C177, C180 to C178, JS3 to JS2, P3 to P1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
Other:
- moved on the sheet: C169, R27, R29
