File: KicadPower/Sensing.kicad_sch (KiCad schematic)
At the start: 11 parts, among them P1 PIN 2, U1 TLE4972-AE35S5

Commit message: readme added and few fixing in schematic and PCB
Parts:
- removed JS2: JumperSMD 3Pin, RezaLIB:JumperSMD 3Pin - UltraSmall, symbol RezaLIB:U_Sensing_2_1_JumperSMD 3Pin_RezaLIB.IntLib
- removed P1: PIN 2, PIN 2, symbol RezaLIB:U_Sensing_2_1_PIN 2_RezaLIB.IntLib
- removed R32: Res SMD, RESC1608X55N, symbol RezaLIB:U_Sensing_2_2_Res SMD_RezaLIB.IntLib
- added J1: Conn_01x03, Connector_PinHeader_2.54mm:PinHeader_1x03_P2.54mm_Vertical, symbol symbols:Conn_01x03
- added R62: 4.7K, Resistor_SMD:R_0603_1608Metric_Pad0.98x0.95mm_HandSolder, symbol Device:R
- added R65: 10R, Resistor_SMD:R_0603_1608Metric_Pad0.98x0.95mm_HandSolder, symbol Device:R
Connections:
- net +3V3_SNS: now also J1.3 (Pin_3), R62.2
- net Iph_P: now also J1.2 (Pin_2)
- net OCD: now also U1.5 (OCD1_N)
- net at C173.2, U1.1 (VDD): now also R65.2
- net at U1.6 (OCD2_N): now also J1.1 (Pin_1), R62.1
- net at FB2.2: now also R65.1
