File: KicadPower/TempSensor.kicad_sch (KiCad schematic)
At the start: 2 parts, among them U17 TMP1075DGKR

Commit message: minor changes
Parts:
- renumbered U17 to U18
Changed lines of the file:
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@@
 		(in_pos_files yes)
 		(dnp no)
-		(property "Reference" "#PWR0113"
+		(property "Reference" "#PWR0112"
 			(at 68.58 96.52 0)
 			(hide yes)
@@
 			(project "MotorDrive_Power"
 				(path "/b3d8444f-9701-4bb0-8db6-84dd09da4106/132a60a0-d8ca-4004-9968-c1990a94735c"
+					(reference "#PWR0112")
+					(unit 1)
+				)
+				(path "/b3d8444f-9701-4bb0-8db6-84dd09da4106/18a84344-2c51-4ad1-a327-06558e4f78c7"
 					(reference "#PWR0113")
-					(unit 1)
-				)
-				(path "/b3d8444f-9701-4bb0-8db6-84dd09da4106/18a84344-2c51-4ad1-a327-06558e4f78c7"
-					(reference "#PWR0112")
 					(unit 1)
 				)
@@
 		(in_pos_files yes)
 		(dnp no)
-		(property "Reference" "U17"
+		(property "Reference" "U18"
 			(at 101.6 91.44 90)
 			(show_name no)
@@
 			(project "MotorDrive_Power"
 				(path "/b3d8444f-9701-4bb0-8db6-84dd09da4106/132a60a0-d8ca-4004-9968-c1990a94735c"
-					(reference "U17")
+					(reference "U18")
 					(unit 1)
 				)
@@
 				)
 				(path "/b3d8444f-9701-4bb0-8db6-84dd09da4106/842552db-c6ca-4109-bc80-82bec330fc23"
-					(reference "U18")
+					(reference "U17")
 					(unit 1)
 				)
@@
 				)
 				(path "/b3d8444f-9701-4bb0-8db6-84dd09da4106/18a84344-2c51-4ad1-a327-06558e4f78c7"
+					(reference "C208")
+					(unit 1)
+				)
+				(path "/b3d8444f-9701-4bb0-8db6-84dd09da4106/842552db-c6ca-4109-bc80-82bec330fc23"
 					(reference "C207")
-					(unit 1)
-				)
-				(path "/b3d8444f-9701-4bb0-8db6-84dd09da4106/842552db-c6ca-4109-bc80-82bec330fc23"
-					(reference "C208")
 					(unit 1)
 				)
@@
 		(in_pos_files yes)
 		(dnp no)
-		(property "Reference" "#PWR0116"
+		(property "Reference" "#PWR0114"
 			(at 68.58 109.22 0)
 			(hide yes)
@@
 			(project "MotorDrive_Power"
 				(path "/b3d8444f-9701-4bb0-8db6-84dd09da4106/132a60a0-d8ca-4004-9968-c1990a94735c"
+					(reference "#PWR0114")
+					(unit 1)
+				)
+				(path "/b3d8444f-9701-4bb0-8db6-84dd09da4106/18a84344-2c51-4ad1-a327-06558e4f78c7"
 					(reference "#PWR0116")
 					(unit 1)
 				)
-				(path "/b3d8444f-9701-4bb0-8db6-84dd09da4106/18a84344-2c51-4ad1-a327-06558e4f78c7"
+				(path "/b3d8444f-9701-4bb0-8db6-84dd09da4106/842552db-c6ca-4109-bc80-82bec330fc23"
 					(reference "#PWR0115")
-					(unit 1)
-				)
-				(path "/b3d8444f-9701-4bb0-8db6-84dd09da4106/842552db-c6ca-4109-bc80-82bec330fc23"
-					(reference "#PWR0114")
 					(unit 1)
 				)
@@
 		(in_pos_files yes)
 		(dnp no)
-		(property "Reference" "#PWR0118"
+		(property "Reference" "#PWR0117"
 			(at 132.08 109.22 0)
 			(hide yes)
@@
 			(project "MotorDrive_Power"
 				(path "/b3d8444f-9701-4bb0-8db6-84dd09da4106/132a60a0-d8ca-4004-9968-c1990a94735c"
+					(reference "#PWR0117")
+					(unit 1)
+				)
+				(path "/b3d8444f-9701-4bb0-8db6-84dd09da4106/18a84344-2c51-4ad1-a327-06558e4f78c7"
 					(reference "#PWR0118")
 					(unit 1)
 				)
-				(path "/b3d8444f-9701-4bb0-8db6-84dd09da4106/18a84344-2c51-4ad1-a327-06558e4f78c7"
-					(reference "#PWR0117")
-					(unit 1)
-				)
