File: KicadPower/TempSensor.kicad_sch (KiCad schematic)
At the start: 2 parts, among them U18 TMP1075DGKR

Commit message: readme added and few fixing in schematic and PCB
Changed lines of the file:
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@@
 	(wire
 		(pts
-			(xy 68.58 109.22) (xy 68.58 106.68)
+			(xy 68.58 106.68) (xy 68.58 110.49)
 		)
 		(stroke
@@
 			(type default)
 			(color 173 188 231 1)
+		)
+	)
+	(wire
+		(pts
+			(xy 132.08 118.11) (xy 132.08 109.22)
+		)
+		(stroke
+			(width 0)
+			(type default)
 		)
 	)
@@
 			)
 			(justify left)
+		)
+	)
+	(symbol
+		(lib_id "symbols:GND")
+		(at 68.58 110.49 0)
+		(unit 1)
+		(body_style 1)
+		(exclude_from_sim no)
+		(in_bom yes)
+		(on_board yes)
+		(in_pos_files yes)
+		(dnp no)
+		(fields_autoplaced yes)
+		(property "Reference" "#PWR0123"
+			(at 68.58 116.84 0)
+			(hide yes)
+			(show_name no)
+			(do_not_autoplace no)
+			(effects
+				(font
+					(size 1.27 1.27)
+				)
+			)
+		)
+		(property "Value" "GND"
+			(at 68.58 115.57 0)
+			(show_name no)
+			(do_not_autoplace no)
+			(effects
+				(font
+					(size 1.27 1.27)
+				)
+			)
+		)
+		(property "Footprint" ""
+			(at 68.58 110.49 0)
+			(hide yes)
+			(show_name no)
+			(do_not_autoplace no)
+			(effects
+				(font
+					(size 1.27 1.27)
+				)
+			)
+		)
+		(property "Datasheet" ""
+			(at 68.58 110.49 0)
+			(hide yes)
+			(show_name no)
+			(do_not_autoplace no)
+			(effects
+				(font
+					(size 1.27 1.27)
+				)
+			)
+		)
+		(property "Description" "Power symbol creates a global label with name \"GND\" , ground"
+			(at 68.58 110.49 0)
+			(hide yes)
+			(show_name no)
+			(do_not_autoplace no)
+			(effects
+				(font
+					(size 1.27 1.27)
+				)
+			)
+		)
+		(pin "1"
+		)
+		(instances
+			(project "MotorDrive_Power"
+				(path "/b3d8444f-9701-4bb0-8db6-84dd09da4106/132a60a0-d8ca-4004-9968-c1990a94735c"
+					(reference "#PWR0123")
+					(unit 1)
+				)
+				(path "/b3d8444f-9701-4bb0-8db6-84dd09da4106/18a84344-2c51-4ad1-a327-06558e4f78c7"
+					(reference "#PWR0125")
+					(unit 1)
+				)
+				(path "/b3d8444f-9701-4bb0-8db6-84dd09da4106/842552db-c6ca-4109-bc80-82bec330fc23"
+					(reference "#PWR0124")
+					(unit 1)
+				)
+			)
 		)
 	)
@@
 	)
 	(symbol
-		(lib_id "MotorDrive_Power-altium-import:GND_POWER_GROUND")
-		(at 68.58 109.22 0)
+		(lib_id "symbols:GND")
+		(at 132.08 118.11 0)
 		(unit 1)
 		(body_style 1)
@@
 		(in_pos_files yes)
 		(dnp no)
-		(property "Reference" "#PWR0114"
-			(at 68.58 109.22 0)
+		(fields_autoplaced yes)
+		(property "Reference" "#PWR0117"
+			(at 132.08 124.46 0)
 			(hide yes)
 			(show_name no)
@@
 		)
 		(property "Value" "GND"
-			(at 68.58 115.57 0)
+			(at 132.08 123.19 0)
 			(show_name no)
 			(do_not_autoplace no)
@@
 		)
 		(property "Footprint" ""
-			(at 68.58 109.22 0)
+			(at 132.08 118.11 0)
+			(hide yes)
 			(show_name no)
 			(do_not_autoplace no)
@@
 		)
 		(property "Datasheet" ""
-			(at 68.58 109.22 0)
-			(show_name no)
-			(do_not_autoplace no)
-			(effects
-				(font
-					(size 1.27 1.27)
-				)
-			)
-		)
-		(property "Description" ""
-			(at 68.58 109.22 0)
-			(show_name no)
-			(do_not_autoplace no)
-			(effects
-				(font
-					(size 1.27 1.27)
-				)
-			)
-		)
-		(pin ""
-		)
-		(instances
-			(project "MotorDrive_Power"
-				(path "/b3d8444f-9701-4bb0-8db6-84dd09da4106/132a60a0-d8ca-4004-9968-c1990a94735c"
-					(reference "#PWR0114")
-					(unit 1)
-				)
-				(path "/b3d8444f-9701-4bb0-8db6-84dd09da4106/18a84344-2c51-4ad1-a327-06558e4f78c7"
-					(reference "#PWR0116")
-					(unit 1)
-				)
-				(path "/b3d8444f-9701-4bb0-8db6-84dd09da4106/842552db-c6ca-4109-bc80-82bec330fc23"
-					(reference "#PWR0115")
-					(unit 1)
-				)
-			)
-		)
-	)
-	(symbol
-		(lib_id "MotorDrive_Power-altium-import:GND_POWER_GROUND")
-		(at 132.08 109.22 0)
-		(unit 1)
-		(body_style 1)
-		(exclude_from_sim no)
-		(in_bom yes)
-		(on_board yes)
-		(in_pos_files yes)
-		(dnp no)
-		(property "Reference" "#PWR0117"
-			(at 132.08 109.22 0)
-			(hide yes)
-			(show_name no)
-			(do_not_autoplace no)
-			(effects
-				(font
-					(size 1.27 1.27)
-				)
-			)
-		)
-		(property "Value" "GND"
-			(at 132.08 115.57 0)
-			(show_name no)
-			(do_not_autoplace no)
-			(effects
-				(font
-					(size 1.27 1.27)
-				)
-			)
-		)
-		(property "Footprint" ""
-			(at 132.08 109.22 0)
-			(show_name no)
-			(do_not_autoplace no)
-			(effects
-				(font
-					(size 1.27 1.27)
-				)
-			)
-		)
-		(property "Datasheet" ""
-			(at 132.08 109.22 0)
-			(show_name no)
-			(do_not_autoplace no)
-			(effects
-				(font
-					(size 1.27 1.27)
-				)
-			)
-		)
-		(property "Description" ""
-			(at 132.08 109.22 0)
-			(show_name no)
-			(do_not_autoplace no)
-			(effects
-				(font
-					(size 1.27 1.27)
-				)
-			)
-		)
-		(pin ""
+			(at 132.08 118.11 0)
+			(hide yes)
+			(show_name no)
+			(do_not_autoplace no)
+			(effects
+				(font
+					(size 1.27 1.27)
+				)
+			)
+		)
+		(property "Description" "Power symbol creates a global label with name \"GND\" , ground"
+			(at 132.08 118.11 0)
+			(hide yes)
+			(show_name no)
+			(do_not_autoplace no)
+			(effects
+				(font
+					(size 1.27 1.27)
+				)
+			)
+		)
+		(pin "1"
 		)
 		(instances
@@
 				)
 				(path "/b3d8444f-9701-4bb0-8db6-84dd09da4106/18a84344-2c51-4ad1-a327-06558e4f78c7"
+					(reference "#PWR0122")
+					(unit 1)
+				)
+				(path "/b3d8444f-9701-4bb0-8db6-84dd09da4106/842552db-c6ca-4109-bc80-82bec330fc23"
 					(reference "#PWR0118")
 					(unit 1)
 				)
-				(path "/b3d8444f-9701-4bb0-8db6-84dd09da4106/842552db-c6ca-4109-bc80-82bec330fc23"
-					(reference "v01")
-					(unit 1)
-				)
