File: KicadPower/Bulk_Caps.kicad_sch (KiCad schematic)
At the start: 144 parts

Commit message: new G serie of Driver modifed and finished
Parts:
- added C185, C186: Cap Pol, CAP-6.3-7.7, symbol RezaLIB:U_PowerStage_2_3_Cap Pol_RezaLIB.IntLib_0
Connections:
- net +Vin: now also C185.1, C186.1
- net PGND: now also C185.2, C186.2

Commit message: changed
Parts:
- removed C16, C185, C186, C19, C22, C7, C8, C9: Cap Pol, CAP-6.3-7.7, symbol RezaLIB:U_PowerStage_2_3_Cap Pol_RezaLIB.IntLib_0
- added C187, C188, C189, C190, C191, C192: 100µF 50V, Capacitor_SMD:C_Elec_8x10.2, symbol Device:C
- added C193, C209: 47µF 50V, Capacitor_SMD:C_Elec_6.3x7.7, symbol Device:C
Connections:
- net +Vin: now also C187.1, C188.1, C189.1, C190.1, C191.1, C192.1, C193.1, C209.1
- net PGND: now also C187.2, C188.2, C189.2, C190.2, C191.2, C192.2, C193.2, C209.2
