File: KicadPower/MotorDrive_Power.kicad_pcb (KiCad board)
At the start: 6 copper layers, 91 x 71 mm, 340 parts, among them IC2 1EDN7116GXTMA1, IC3 1EDN7116GXTMA1, IC4 1EDN7116GXTMA1, IC5 1EDN7116GXTMA1, IC6 1EDN7116GXTMA1, IC7 1EDN7116GXTMA1, P1 PIN 2, P2 PIN 2, P3 PIN 2, P4 Connector, P5 Connector, P6 Header 20X2, P7 Connector, P8 Connector, P9 Connector, Q1 IGB110S101, Q10 IGB110S101, Q11 IGB110S101, Q12 IGB110S101, Q13 IGB110S101, Q14 IGB110S101, Q15 IGB110S101, Q16 IGB110S101, Q17 IGB110S101, Q18 IGB110S101, Q19 IGB110S101, Q2 IGB110S101, Q20 IGB110S101, Q21 IGB110S101, Q22 IGB110S101, Q23 IGB110S101, Q24 IGB110S101, Q3 IGB110S101, Q4 IGB110S101, Q5 IGB110S101, Q6 IGB110S101, Q7 IGB110S101, Q8 IGB110S101, Q9 IGB110S101, U1 TLE4972-AE35S5, U10 LDK220C-R, U17 TMP1075DGKR, U18 TMP1075DGKR, U19 TMP1075DGKR, U2 TLE4972-AE35S5, U3 TLE4972-AE35S5, U4 LDK220C-R, U5 LDK220C, U6 LDK220C, U7 LDK220C, U8 LDK220C-R, U9 LDK220C-R

Commit message: changed
Parts:
- removed C16, C185, C186, C19, C22, C7, C8, C9: Cap Pol, RezaLIB:CAP-6.3-7.7
- added ?: , , F.Cu at (190.0, 136.5)
- added ?: , , F.Cu at (162.5, 72.4)
- added ?: , , F.Cu at (107.0, 136.5)
- added ?: , , F.Cu at (132.2, 72.4)
- added C187: 100µF 50V, Capacitor_SMD:C_Elec_8x10.2, F.Cu at (167.7, 78.5)
- added C188: 100µF 50V, Capacitor_SMD:C_Elec_8x10.2, F.Cu at (157.7, 78.5)
- added C189: 100µF 50V, Capacitor_SMD:C_Elec_8x10.2, F.Cu at (137.5, 78.5)
- added C190: 100µF 50V, Capacitor_SMD:C_Elec_8x10.2, F.Cu at (127.2, 78.5)
- added C191: 100µF 50V, Capacitor_SMD:C_Elec_8x10.2, F.Cu at (107.4, 78.5)
- added C192: 100µF 50V, Capacitor_SMD:C_Elec_8x10.2, F.Cu at (189.5, 78.5)
- added C193: 47µF 50V, Capacitor_SMD:C_Elec_6.3x7.7, F.Cu at (107.1, 129.3)
- added C209: 47µF 50V, Capacitor_SMD:C_Elec_6.3x7.7, F.Cu at (189.3, 129.4)
- moved FB1 0.42 mm to (111.5, 79.1)
- moved R61 0.25 mm to (118.5, 100.2)
- moved C150 0.25 mm to (192.5, 96.8)
- moved FB4 0.15 mm to (181.3, 110.0)
- moved D5 0.15 mm to (117.6, 104.3)
- moved FB3 0.09 mm to (142.3, 78.7)
Routing:
- net +10V: track 197.2 -> 190.9 mm
- net GND: track 52.4 -> 57.8 mm, vias 42 -> 54
- net /OCD: track 142.8 -> 138.7 mm
- net Net-(U1-OCD2_N): track 15.7 -> 13.0 mm
- net Net-(U2-OCD2_N): track 14.1 -> 16.2 mm
- net Net-(U3-OCD2_N): track 14.7 -> 16.7 mm
- net /IP_P3: track 79.5 -> 77.6 mm
- net +Vin: track 16.1 -> 14.2 mm, vias 463 -> 472
- net /Phase_S: track 33.7 -> 32.0 mm, vias 90 -> 93
- net +3V3_SNS: track 74.7 -> 73.6 mm
- net +3V3: track 161.0 -> 160.0 mm
- net Net-(IC3-IN+): track 40.3 -> 41.2 mm
- net /IP_N3: track 80.2 -> 79.4 mm
- net Net-(U1-OCD1_N): track 4.78 -> 4.18 mm
- net PGND: vias 565 -> 578
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Other:
- board text added: "Reza Sede"
- board text added: "eGAN FET Motor Controller V1.0"
