File: KicadPower/MotorDrive_Power.kicad_pcb (KiCad board)
At the start: 6 copper layers, 91 x 71 mm, 344 parts, among them IC2 1EDN7116GXTMA1, IC3 1EDN7116GXTMA1, IC4 1EDN7116GXTMA1, IC5 1EDN7116GXTMA1, IC6 1EDN7116GXTMA1, IC7 1EDN7116GXTMA1, P1 PIN 2, P2 PIN 2, P3 PIN 2, P4 Connector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

Commit message: Sent for Manufacturing V1.0
Other:
- board text added: "V1.0"
- board text added: "eGAN FET Motor Controller Power Section"
- board text removed: "eGAN FET Motor Controller V1.0"
