File: KicadPower/Connector.kicad_sch (KiCad schematic)
At the start: 8 parts, among them P6 Header 20X2, U4 LDK220C-R

Commit message: readme added and few fixing in schematic and PCB
Connections:
- net +Vin: no longer P6.37
- new net +3V3: P6.37
Changed lines of the file:
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@@
-	)
-	(junction
-		(at 114.3 121.1072)
-		(diameter 0)
-		(color 0 0 0 0)
 	)
 	(junction
@@
 	(wire
 		(pts
+			(xy 114.3 118.11) (xy 114.3 118.5672)
+		)
+		(stroke
+			(width 0)
+			(type default)
+		)
+	)
+	(wire
+		(pts
 			(xy 114.3 116.0272) (xy 114.3 113.4872)
 		)
@@
 	(wire
 		(pts
+			(xy 106.68 118.11) (xy 114.3 118.11)
+		)
+		(stroke
+			(width 0)
+			(type default)
+		)
+	)
+	(wire
+		(pts
 			(xy 69.85 179.5272) (xy 78.74 179.5272)
 		)
@@
 	(wire
 		(pts
-			(xy 114.3 121.1072) (xy 114.3 118.5672)
-		)
-		(stroke
-			(width 0)
-			(type default)
-		)
-	)
-	(wire
-		(pts
 			(xy 147.32 108.4072) (xy 134.62 108.4072)
 		)
@@
 		(pts
 			(xy 233.68 103.3272) (xy 223.52 103.3272)
+		)
+		(stroke
+			(width 0)
+			(type default)
+		)
+	)
+	(wire
+		(pts
+			(xy 106.68 114.3) (xy 106.68 118.11)
 		)
 		(stroke
@@
 					(unit 1)
 				)
+			)
+		)
+	)
+	(symbol
+		(lib_id "MotorDrive_Power-altium-import:+3V3_BAR")
+		(at 106.68 114.3 180)
+		(unit 1)
+		(body_style 1)
+		(exclude_from_sim no)
+		(in_bom yes)
+		(on_board yes)
+		(in_pos_files yes)
+		(dnp no)
+		(property "Reference" "#PWR0121"
+			(at 106.68 114.3 0)
+			(hide yes)
+			(show_name no)
+			(do_not_autoplace no)
+			(effects
+				(font
+					(size 1.27 1.27)
+				)
+			)
+		)
+		(property "Value" "+3V3"
+			(at 106.68 110.49 0)
+			(show_name no)
+			(do_not_autoplace no)
+			(effects
+				(font
+					(size 1.27 1.27)
+				)
+			)
+		)
+		(property "Footprint" ""
+			(at 106.68 114.3 0)
+			(show_name no)
+			(do_not_autoplace no)
+			(effects
+				(font
+					(size 1.27 1.27)
+				)
+			)
+		)
+		(property "Datasheet" ""
+			(at 106.68 114.3 0)
+			(show_name no)
+			(do_not_autoplace no)
+			(effects
+				(font
+					(size 1.27 1.27)
+				)
+			)
+		)
+		(property "Description" ""
+			(at 106.68 114.3 0)
+			(show_name no)
+			(do_not_autoplace no)
+			(effects
+				(font
+					(size 1.27 1.27)
+				)
+			)
+		)
+		(pin ""
+		)
+		(instances
+			(project "MotorDrive_Power"
+				(path "/b3d8444f-9701-4bb0-8db6-84dd09da4106/9252f410-1898-4564-9d05-e8bcb0be908b"
+					(reference "#PWR0121")
+					(unit 1)
+				)
