File: KicadPower/GateDrive.kicad_sch (KiCad schematic)
At the start: 22 parts, among them IC2 1EDN7116GXTMA1, IC5 1EDN7116GXTMA1, U7 LDK220C, U8 LDK220C-R

Commit message: readme added and few fixing in schematic and PCB
Parts:
- removed D3, D6: SS34, DO-214AC, symbol RezaLIB:U_GateDrive_1_Generic Diode_RezaLIB.IntLib
- added D17, D20, D23: SS34, Diode_SMD:D_SMA, symbol symbols:SS34
Connections:
- net at C212.1, R41.2, U8.1 (IN)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: now also D23.2 (A)
- net at C194.1, C200.1, D10.1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: now also D20.1 (K)
- net at R59.2: now also D20.2 (A)
- net at R56.2: now also D17.1 (K); no longer IC2.7 (BST)
- net at C215.1, U7.1 (IN), U7.3 (EN): now also D23.1 (K)
- new net: D17.2 (A), IC2.7 (BST)
