File: KicadControlAURIX/Control.kicad_sch (KiCad schematic)
At the start: 64 parts, among them P1 PIN 4, P2 Header 20X2, P3 Connector, P4 Header 20X2, P5 Connector, P6 Header 20X2

Commit message: changed
Parts:
- added C25: 1uF, Capacitor_SMD:C_0805_2012Metric_Pad1.18x1.45mm_HandSolder, symbol Device:C
Connections:
- net +10V: now also P5.5, C25.2
- net +5V: no longer P5.5
- net GND: now also C25.1
Other:
- moved on the sheet: C1, C10, C11, C12, C13, C14, C15, C16, C2, C3, C4, C5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
