File: KicadControlAURIX/PSU.kicad_sch (KiCad schematic)
At the start: 38 parts, among them P7 Power jack, U1 LDK220C-R

Commit message: changed
Parts:
- removed C17: Cap Pol, CAP-4.0-5.3, symbol RezaLIB:U_PSU_3_Cap Pol_RezaLIB.IntLib_0
- added C24: 47µF 50V, Capacitor_SMD:C_Elec_6.3x7.7, symbol Device:C
- added C26: 220µF 16V, Capacitor_SMD:C_Elec_6.3x7.7, symbol Device:C
Connections:
- net +10V: now also C26.1
- net +Vin: now also C24.1
- net GND: now also C24.2, C26.2
Other:
- moved on the sheet: D1
