File: KicadControlAURIX/MotorDrive_Control_AURIX.kicad_pcb (KiCad board)
At the start: 2 copper layers, 95 x 100 mm, 112 parts, among them P1 PIN 4, P2 Header 20X2, P3 Connector, P4 Header 20X2, P5 Connector, P6 Header 20X2, P7 Power jack, U1 LDK220C-R

Commit message: changed
Parts:
- removed C17: Cap Pol, RezaLIB:CAP-4.0-5.3
- added C24: 47µF 50V, Capacitor_SMD:C_Elec_6.3x7.7, F.Cu at (168.3, 86.3)
- added C25: 1uF, Capacitor_SMD:C_0805_2012Metric_Pad1.18x1.45mm_HandSolder, F.Cu at (190.9, 100.5)
- added C26: 220µF 16V, Capacitor_SMD:C_Elec_6.3x7.7, F.Cu at (190.8, 81.0)
Connections:
- P5 pad 5: +5V -> +10V
Routing:
- net +10V: track 170.8 -> 176.6 mm
- net GND: vias 346 -> 348
Other:
- board text added: "AURIX TC4D Processor KIT_A3G_TC4D7_LITE SAKTC4D7XP-20MF500MC AA"
- board text added: "Debug"
- board text added: "Encoder"
- board text added: "HAL"
- board text added: "Reza Sede AURIX Motor Controller V1.0"
- board text removed: "B"

Commit message: Sent for Manufacturing V1.0
Other:
- board text added: "Reza Sede"
- board text added: "V1.0"
- board text added: "eGAN FET Motor Controller Control Section"
- board text removed: "Reza Sede AURIX Motor Controller V1.0"
